File: OpenRectangle.kicad_pcb (KiCad board)
At the start: 2 copper layers, 21 parts, among them J1 RPI_PICO-TH, SW1 MX_SW_HS, SW10 MX_SW_HS, SW11 MX_SW_HS, SW12 MX_SW_HS, SW13 MX_SW_HS, SW14 MX_SW_HS, SW15 MX_SW_HS, SW16 MX_SW_HS, SW17 MX_SW_HS, SW18 MX_SW_HS, SW19 MX_SW_HS, SW2 MX_SW_HS, SW20 MX_SW_HS, SW3 MX_SW_HS, SW4 MX_SW_HS, SW5 MX_SW_HS, SW6 MX_SW_HS, SW7 MX_SW_HS, SW8 MX_SW_HS, SW9 MX_SW_HS

Commit message: Técnicamente ya funciona
Parts:
- added D1: D_Small, Diode_THT:D_DO-41_SOD81_P10.16mm_Horizontal, F.Cu at (193.7, 51.6)
- added D2: D_Small, Diode_SMD:D_0805_2012Metric, F.Cu at (199.2, 51.6)
- added J1: Left Stick, Connector_PinHeader_2.54mm:PinHeader_1x05_P2.54mm_Vertical, F.Cu at (105.0, 74.9)
- added J10: Modifiers, Connector_PinHeader_2.54mm:PinHeader_1x03_P2.54mm_Vertical, F.Cu at (161.6, 86.5)
- added J11: C Stick, Connector_PinHeader_2.54mm:PinHeader_1x06_P2.54mm_Vertical, F.Cu at (170.6, 122.2)
- added J12: Buttons, Connector_PinHeader_2.54mm:PinHeader_1x09_P2.54mm_Vertical, F.Cu at (192.4, 110.2)
- added J2: Buttons, Connector_PinHeader_2.54mm:PinHeader_1x09_P2.54mm_Vertical, F.Cu at (315.7, 74.6)
- added J3: Modifiers, Connector_PinHeader_2.54mm:PinHeader_1x03_P2.54mm_Vertical, F.Cu at (142.7, 145.6)
- added J4: C Stick, Connector_PinHeader_2.54mm:PinHeader_1x06_P2.54mm_Vertical, F.Cu at (238.4, 147.7)
- added J5: GCC Cable, Connector_PinHeader_2.54mm:PinHeader_1x06_P2.54mm_Vertical, F.Cu at (176.2, 30.2)
- added J6: Extra USB, Connector_PinHeader_2.54mm:PinHeader_1x04_P2.54mm_Vertical, F.Cu at (180.9, 53.5)
- added J7: USB C Connector, Connector_USB:USB_C_Receptacle_Amphenol_12401548E4-2A, F.Cu at (198.6, 29.4)
- added J9: Left Stick, Connector_PinHeader_2.54mm:PinHeader_1x05_P2.54mm_Vertical, F.Cu at (161.6, 70.7)
- moved SW8 590.1 mm to (92.3, 62.6)
- moved SW15 558.5 mm to (148.5, 157.2)
- moved SW14 536.6 mm to (125.8, 141.5)
- moved SW9 503.0 mm to (118.8, 74.3)
- moved SW5 423.4 mm to (198.6, 74.3)
- moved SW20 413.5 mm to (293.3, 126.1)
- moved SW1 412.7 mm to (277.6, 46.3)
- moved SW2 409.0 mm to (304.2, 34.3)
- moved SW18 397.3 mm to (247.9, 157.2)
- moved SW10 384.6 mm to (277.6, 74.0)
- moved SW16 374.4 mm to (247.9, 126.1)
- moved SW19 371.7 mm to (270.6, 141.5)
- moved SW11 358.9 mm to (304.2, 62.0)
- moved SW12 350.5 mm to (332.5, 64.9)
- moved SW17 333.9 mm to (270.6, 110.3)
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- renumbered J1 to J8, SW16 to SW14, SW17 to SW15, SW14 to SW16, SW15 to SW17
Connections:
- J8 pad AGND: unconnected-(J1-PadAGND) -> GND
- J8 pad GND@1: Net-(J1-PadGND@1) -> GND
- J8 pad GND@2: Net-(J1-PadGND@1) -> GND
- J8 pad GND@3: Net-(J1-PadGND@1) -> GND
- J8 pad GND@4: Net-(J1-PadGND@1) -> GND
- J8 pad GND@5: Net-(J1-PadGND@1) -> GND
- J8 pad GND@6: Net-(J1-PadGND@1) -> GND
- J8 pad GND@7: Net-(J1-PadGND@1) -> GND
- J8 pad GND@8: Net-(J1-PadGND@1) -> GND
- J8 pad GP0: unconnected-(J1-PadGP0) -> P START
- J8 pad GP12: unconnected-(J1-PadGP12) -> P C_UP
- J8 pad GP13: unconnected-(J1-PadGP13) -> P C_LT
- J8 pad GP14: unconnected-(J1-PadGP14) -> P A
- J8 pad GP15: unconnected-(J1-PadGP15) -> P C_DN
- J8 pad GP16: unconnected-(J1-PadGP16) -> P C_RT
- J8 pad GP17: unconnected-(J1-PadGP17) -> P UP
- J8 pad GP18: unconnected-(J1-PadGP18) -> P MS
- J8 pad GP19: unconnected-(J1-PadGP19) -> P Z
- J8 pad GP2: unconnected-(J1-PadGP2) -> P RIGHT
- J8 pad GP20: unconnected-(J1-PadGP20) -> P LS
- J8 pad GP21: unconnected-(J1-PadGP21) -> P X
- J8 pad GP22: unconnected-(J1-PadGP22) -> P Y
- J8 pad GP26_A0: unconnected-(J1-PadGP26_A0) -> P B
- J8 pad GP27_A1: unconnected-(J1-PadGP27_A1) -> P R
- J8 pad GP28_A2: unconnected-(J1-PadGP28_A2) -> DATA
- J8 pad GP3: unconnected-(J1-PadGP3) -> P DOWN
- J8 pad GP4: unconnected-(J1-PadGP4) -> P LEFT
- J8 pad GP5: unconnected-(J1-PadGP5) -> P L
- J8 pad GP6: unconnected-(J1-PadGP6) -> P M1
- J8 pad GP7: unconnected-(J1-PadGP7) -> P M2
- J8 pad TP2: unconnected-(J1-PadTP2) -> D-
- J8 pad TP3: unconnected-(J1-PadTP3) -> D+
- J8 pad VBUS: unconnected-(J1-PadVBUS) -> +5V
- J8 pad VSYS: unconnected-(J1-PadVSYS) -> VCC
- SW1 pad 1: unconnected-(SW1-Pad1) -> GND
- SW1 pad 2: unconnected-(SW1-Pad2) -> R
- SW10 pad 1: unconnected-(SW10-Pad1) -> GND
- SW10 pad 2: unconnected-(SW10-Pad2) -> B
- SW11 pad 1: unconnected-(SW11-Pad1) -> GND
- SW11 pad 2: unconnected-(SW11-Pad2) -> X
- SW12 pad 1: unconnected-(SW12-Pad1) -> GND
- SW12 pad 2: unconnected-(SW12-Pad2) -> Z
- SW13 pad 1: unconnected-(SW13-Pad1) -> GND
- SW13 pad 2: unconnected-(SW13-Pad2) -> UP
- SW14 pad 1: unconnected-(SW16-Pad1) -> GND
- SW14 pad 2: unconnected-(SW16-Pad2) -> M1
- SW15 pad 1: unconnected-(SW17-Pad1) -> GND
- SW15 pad 2: unconnected-(SW17-Pad2) -> M2
- SW16 pad 1: unconnected-(SW14-Pad1) -> GND
- SW16 pad 2: unconnected-(SW14-Pad2) -> C_LT
- SW17 pad 1: unconnected-(SW15-Pad1) -> GND
- SW17 pad 2: unconnected-(SW15-Pad2) -> C_UP
- SW18 pad 1: unconnected-(SW18-Pad1) -> GND
- SW18 pad 2: unconnected-(SW18-Pad2) -> C_DN
- SW19 pad 1: unconnected-(SW19-Pad1) -> GND
- SW19 pad 2: unconnected-(SW19-Pad2) -> A
- SW2 pad 1: unconnected-(SW2-Pad1) -> GND
- SW2 pad 2: unconnected-(SW2-Pad2) -> Y
- SW20 pad 1: unconnected-(SW20-Pad1) -> GND
- SW20 pad 2: unconnected-(SW20-Pad2) -> C_RT
- SW3 pad 1: unconnected-(SW3-Pad1) -> GND
- SW3 pad 2: unconnected-(SW3-Pad2) -> LS
- SW4 pad 1: unconnected-(SW4-Pad1) -> GND
- SW4 pad 2: unconnected-(SW4-Pad2) -> MS
- SW5 pad 1: unconnected-(SW5-Pad1) -> GND
- SW5 pad 2: unconnected-(SW5-Pad2) -> START
- SW6 pad 2: unconnected-(SW6-Pad2) -> L
- SW7 pad 2: unconnected-(SW7-Pad2) -> LEFT
- SW8 pad 2: unconnected-(SW8-Pad2) -> DOWN
- SW9 pad 2: unconnected-(SW9-Pad2) -> RIGHT
Routing:
- net +5V: track 0.00 -> 108.4 mm
- net A: track 0.00 -> 95.7 mm
- net DATA: track 0.00 -> 92.9 mm
- net VCC: track 0.00 -> 90.7 mm
- net C_UP: track 0.00 -> 84.9 mm
- net MS: track 0.00 -> 80.9 mm
- net Y: track 0.00 -> 74.8 mm
- net LS: track 0.00 -> 72.1 mm
- net +3V3: track 0.00 -> 63.6 mm
- net C_RT: track 0.00 -> 62.7 mm
- net UP: track 0.00 -> 52.5 mm
- net L: track 0.00 -> 50.6 mm
- net D-: track 0.00 -> 47.5 mm, vias 0 -> 1
- net Z: track 0.00 -> 45.8 mm
- net D+: track 0.00 -> 44.1 mm
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- added copper zone on B.Cu, net GND
- added copper zone on F.Cu, net GND
Other:
- board outline added: 339.1 x 142 mm
