File: OpenRectangle.kicad_pcb (KiCad board)
At the start: 2 copper layers, 339.1 x 141.2 mm, 54 parts, among them J1 USB C Connector, J2 GCC Cable, J3 JTAG_TC2030, SW1 MX_SW_HS, SW10 MX_SW_HS, SW11 MX_SW_HS, SW12 MX_SW_HS, SW13 MX_SW_HS, SW14 MX_SW_HS, SW15 MX_SW_HS, SW16 MX_SW_HS, SW17 MX_SW_HS, SW18 MX_SW_HS, SW19 MX_SW_HS, SW2 MX_SW_HS, SW20 MX_SW_HS, SW21 Boot, SW3 MX_SW_HS, SW4 MX_SW_HS, SW5 MX_SW_HS, SW6 MX_SW_HS, SW7 MX_SW_HS, SW8 MX_SW_HS, SW9 MX_SW_HS, U1 XC6206, U2 USBLC6-2SC6, U3 RP2040, U4 W25Q128JVS, Y1 12MHz

Commit message: Holy shit man
Parts:
- removed J2: GCC Cable, Connector_PinHeader_2.54mm:PinHeader_1x06_P2.54mm_Vertical
- removed R1, R2: 5.1k, Resistor_SMD:R_0402_1005Metric
- added F1: Fuse_Small, Fuse:Fuse_1206_3216Metric, F.Cu at (202.4, 38.1)
- D1: value D_Small -> Schottky Diode; footprint Diode_SMD:D_0805_2012Metric -> qw-footprints:CUSTOM D_SOD-123
- J1: footprint Connector_USB:USB_C_Receptacle_Amphenol_12401548E4-2A -> qw-footprints:TYPE-C_24P_QCHT
- moved U3 139.8 mm to (198.6, 54.9)
- moved J3 131.1 mm to (208.9, 69.8), turned to 180 degrees
- moved Y1 124.1 mm to (196.3, 66.0), turned to 180 degrees
- moved R7 123.0 mm to (191.8, 33.3)
- moved R3 120.6 mm to (209.8, 65.2), turned to 180 degrees
- moved C9 117.3 mm to (202.4, 48.7), turned to 90 degrees
- moved C11 115.5 mm to (199.5, 62.5), turned to -90 degrees
- moved C15 113.7 mm to (192.9, 66.3), turned to -90 degrees
- moved C16 112.6 mm to (199.6, 66.1), turned to 90 degrees
- moved SW21 112.3 mm to (182.2, 30.2)
- moved C12 111.8 mm to (192.3, 57.0), turned to -135 degrees
- moved C4 111.1 mm to (197.1, 46.9), turned to 90 degrees
- moved C14 110.8 mm to (205.1, 51.4)
- moved R6 109.2 mm to (197.4, 62.5), turned to 90 degrees
- moved C8 109.1 mm to (205.9, 57.8), turned to -45 degrees
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Connections:
- J1 pad A4: +5V -> Net-(J1-PadA4)
- J1 pad A9: +5V -> Net-(J1-PadA4)
- J1 pad B4: +5V -> Net-(J1-PadA4)
- J1 pad B9: +5V -> Net-(J1-PadA4)
- U2 pad 1: DBUS- -> DBUS+
- U2 pad 3: DBUS+ -> DBUS-
- U2 pad 4: D+ -> D-
- U2 pad 6: D- -> D+
Routing:
- net +3V3: track 0.00 -> 67.6 mm, vias 0 -> 3
- net GND: track 0.00 -> 51.9 mm, vias 0 -> 16
- net CS: track 0.00 -> 32.2 mm
- net +1V1: track 0.00 -> 28.9 mm, vias 0 -> 5
- net SD1: track 0.00 -> 28.6 mm
- net SD2: track 0.00 -> 23.4 mm
- net SD0: track 0.00 -> 14.8 mm
- net XTAL_IN: track 0.00 -> 14.3 mm
- net QSPI_CLK: track 0.00 -> 14.0 mm
- net SD3: track 0.00 -> 13.6 mm
- net unconnected-(U3-Pad41): track 0.00 -> 11.8 mm
- net DATA: track 0.00 -> 11.3 mm
- net SWD: track 0.00 -> 10.8 mm
- net SWCLK: track 0.00 -> 10.8 mm
- net R: track 0.00 -> 10.8 mm
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- added copper zone on F.Cu, net +1V1
- added copper zone on F.Cu, net +3V3
- added copper zone on B.Cu, net GND
- added copper zone on F.Cu, net GND
Other:
- board text added: "100nF"
- board text added: "RP2040"
