File: OpenRectangle.kicad_pcb (KiCad board)
At the start: 2 copper layers, 339.1 x 141.2 mm, 85 parts, among them J1 USB C Connector, J2 JTAG_TC2030, SW1 MX_SW_HS, SW10 MX_SW_HS, SW11 MX_SW_HS, SW12 MX_SW_solder, SW13 MX_SW_HS, SW14 MX_SW_solder, SW15 MX_SW_solder, SW16 MX_SW_HS, SW17 MX_SW_HS, SW18 MX_SW_solder, SW19 MX_SW_HS, SW2 MX_SW_solder, SW20 MX_SW_solder, SW21 MX_SW_solder, SW22 MX_SW_HS, SW23 MX_SW_HS, SW24 MX_SW_solder, SW25 MX_SW_solder, SW26 MX_SW_HS, SW27 MX_SW_solder, SW28 MX_SW_HS, SW29 MX_SW_HS, SW3 MX_SW_HS, SW30 MX_SW_solder, SW31 MX_SW_solder, SW32 MX_SW_HS, SW33 MX_SW_solder, SW34 MX_SW_HS, SW35 MX_SW_HS, SW36 MX_SW_solder, SW37 MX_SW_solder, SW38 MX_SW_HS, SW39 MX_SW_HS, SW4 MX_SW_solder, SW40 MX_SW_solder, SW41 Boot, SW5 MX_SW_HS, SW6 MX_SW_solder, SW7 MX_SW_HS, SW8 MX_SW_solder, SW9 MX_SW_solder, U1 XC6206, U2 USBLC6-2SC6, U3 RP2040, U4 W25Q128JVS, Y1 12MHz

Commit message: Updates version
Added:
- C to C functionality
- VBUS sensing
- Green LED
- Shield connected to GND via a resistor
Parts:
- removed the SW1 at (198.6, 94.3)
- added D3: GREEN, LED_SMD:LED_0805_2012Metric, F.Cu at (211.0, 53.5)
- added R1: 1M, Resistor_SMD:R_0603_1608Metric, F.Cu at (205.7, 26.7)
- added R2: 5.1k, Resistor_SMD:R_0402_1005Metric, F.Cu at (194.4, 35.2)
- added R3: 5.1k, Resistor_SMD:R_0402_1005Metric, F.Cu at (205.3, 32.6)
- added R4: 470, Resistor_SMD:R_0402_1005Metric, F.Cu at (208.3, 53.5)
- added R5: 5.6k, Resistor_SMD:R_0603_1608Metric, F.Cu at (209.0, 49.6)
- added R6: 10k, Resistor_SMD:R_0603_1608Metric, F.Cu at (210.6, 49.6)
- added SW41: MX_SW_solder, marbastlib-mx:SW_MX_1u, F.Cu at (293.3, 126.1)
- F1: value Fuse_Small -> 500 mA
- R8: renamed from R2; value 27R -> 27
- R9: renamed from R3; value 27R -> 27
- SW10, SW17, SW19, SW23, SW29, SW3, SW35, SW38, SW7: value MX_SW_HS -> MX_SW_solder; footprint marbastlib-mx:SW_MX_HS_1u -> marbastlib-mx:SW_MX_1u; moved to F.Cu
- SW14, SW18, SW2, SW21, SW24, SW31, SW36, SW40, SW6, SW9: value MX_SW_solder -> MX_SW_HS; footprint marbastlib-mx:SW_MX_1u -> marbastlib-mx:SW_MX_HS_1u; moved to B.Cu
- moved SW27 240.7 mm to (358.7, 81.0)
- moved SW11 161.2 mm to (118.8, 74.3)
- moved SW3 160.4 mm to (198.6, 94.3)
- moved SW31 104.2 mm to (148.5, 157.2)
- moved SW19 83.7 mm to (358.7, 53.4)
- moved SW35 52.1 mm to (270.6, 110.3)
- moved SW17 30.7 mm to (332.5, 37.3)
- moved SW25 30.7 mm to (332.5, 64.9)
- moved SW5 30.1 mm to (38.6, 81.6)
- moved SW13 29.1 mm to (277.6, 46.3)
- moved SW21 29.1 mm to (277.6, 74.0)
- moved SW9 29.1 mm to (92.3, 62.5)
- moved SW15 28.5 mm to (304.2, 34.3)
- moved SW23 28.5 mm to (304.2, 62.0)
- moved SW7 28.5 mm to (63.9, 65.3)
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- renumbered C7 to C10, C8 to C11, C9 to C12, C10 to C13, C11 to C14, C12 to C15, C13 to C16, C14 to C17, C17 to C3, C3 to C4, C4 to C5, C5 to C6, C15 to C7, C16 to C8, C6 to C9, D2 to D1, D1 to D2, H11 to H1, H7 to H10, H8 to H11, H1 to H2, H2 to H3, H3 to H4, H4 to H5, H9 to H6, H5 to H7, H6 to H8, H10 to H9, R5 to R10, R4 to R11, R1 to R7, SW41 to SW1
Connections:
- net VCC renamed Net-(F1-Pad1)
- J1 pad A5: unconnected-(J1-PadA5) -> Net-(J1-CC1)
- J1 pad B5: unconnected-(J1-PadB5) -> Net-(J1-CC2)
- J1 pad S1: GND -> Net-(J1-SHIELD)
- SW10 pad 1: GND -> RIGHT
- SW10 pad 2: RIGHT -> GND
- SW11 pad 2: R -> RIGHT
- SW13 pad 2: Y -> R
- SW14 pad 1: Y -> GND
- SW14 pad 2: GND -> Y
- SW15 pad 1: LS -> Y
- SW17 pad 1: GND -> LS
- SW17 pad 2: MS -> GND
- SW18 pad 1: MS -> GND
- SW18 pad 2: GND -> MS
- SW19 pad 1: GND -> MS
- SW19 pad 2: B -> GND
- SW2 pad 1: START -> GND
- SW2 pad 2: GND -> START
- SW21 pad 1: X -> GND
- SW21 pad 2: GND -> B
- SW23 pad 1: GND -> X
- SW23 pad 2: Z -> GND
- SW24 pad 1: Z -> GND
- SW24 pad 2: GND -> Z
- SW25 pad 1: UP -> Z
- SW27 pad 1: M1 -> UP
- SW29 pad 1: GND -> M1
- SW29 pad 2: M2 -> GND
- SW3 pad 1: GND -> START
- SW3 pad 2: L -> GND
- SW31 pad 1: C_LT -> GND
- SW31 pad 2: GND -> M2
- SW33 pad 1: C_UP -> C_LT
- SW35 pad 1: GND -> C_UP
- SW35 pad 2: C_DN -> GND
- SW36 pad 1: C_DN -> GND
- SW36 pad 2: GND -> C_DN
- SW37 pad 1: A -> C_DN
- SW38 pad 1: GND -> A
- SW38 pad 2: A -> GND
- SW39 pad 2: C_RT -> A
- SW40 pad 1: C_RT -> GND
- SW40 pad 2: GND -> C_RT
- SW5 pad 2: LEFT -> L
- SW6 pad 1: LEFT -> GND
- SW6 pad 2: GND -> LEFT
- SW7 pad 1: GND -> LEFT
- SW7 pad 2: DOWN -> GND
- SW9 pad 1: RIGHT -> GND
- SW9 pad 2: GND -> DOWN
- U3 pad 2: START -> unconnected-(U3-GPIO0-Pad2)
- U3 pad 3: unconnected-(U3-Pad3) -> START
- U3 pad 35: unconnected-(U3-Pad35) -> B
- U3 pad 36: unconnected-(U3-Pad36) -> R
- U3 pad 38: B -> unconnected-(U3-GPIO26/ADC0-Pad38)
- U3 pad 39: R -> PICO_LED
- U3 pad 40: DATA -> VBUS_SENSE
- U3 pad 41: unconnected-(U3-Pad41) -> DATA
Routing:
- net Net-(J1-SHIELD): track 0.00 -> 23.5 mm
- net +5V: track 10.6 -> 30.4 mm
- net Net-(J1-CC2): track 0.00 -> 15.6 mm
- net VBUS_SENSE: track 0.00 -> 10.6 mm
- net Net-(J1-CC1): track 0.00 -> 9.91 mm, vias 0 -> 2
- net PICO_LED: track 0.00 -> 5.81 mm
- net Net-(D3-A): track 0.00 -> 1.18 mm
- net Net-(D1-A): track 1.72 -> 2.61 mm
