File: OpenRectangle.kicad_sch (KiCad schematic)
At the start: 21 parts, among them J1 RPI_PICO-TH, SW1 MX_SW_HS, SW10 MX_SW_HS, SW11 MX_SW_HS, SW12 MX_SW_HS, SW13 MX_SW_HS, SW14 MX_SW_HS, SW15 MX_SW_HS, SW16 MX_SW_HS, SW17 MX_SW_HS, SW18 MX_SW_HS, SW19 MX_SW_HS, SW2 MX_SW_HS, SW20 MX_SW_HS, SW3 MX_SW_HS, SW4 MX_SW_HS, SW5 MX_SW_HS, SW6 MX_SW_HS, SW7 MX_SW_HS, SW8 MX_SW_HS, SW9 MX_SW_HS

Commit message: Técnicamente ya funciona
Parts:
- added D1: D_Small, Diode_THT:D_DO-41_SOD81_P10.16mm_Horizontal, symbol Device:D_Small
- added D2: D_Small, Diode_SMD:D_0805_2012Metric, symbol Device:D_Small
- added J1, J9: Left Stick, Connector_PinHeader_2.54mm:PinHeader_1x05_P2.54mm_Vertical, symbol Connector:Conn_01x05_Male
- added J10, J3: Modifiers, Connector_PinHeader_2.54mm:PinHeader_1x03_P2.54mm_Vertical, symbol Connector:Conn_01x03_Male
- added J11, J4: C Stick, Connector_PinHeader_2.54mm:PinHeader_1x06_P2.54mm_Vertical, symbol Connector:Conn_01x06_Male
- added J12, J2: Buttons, Connector_PinHeader_2.54mm:PinHeader_1x09_P2.54mm_Vertical, symbol Connector:Conn_01x09_Male
- added J5: GCC Cable, Connector_PinHeader_2.54mm:PinHeader_1x06_P2.54mm_Vertical, symbol Connector:Conn_01x06_Female
- added J6: Extra USB, Connector_PinHeader_2.54mm:PinHeader_1x04_P2.54mm_Vertical, symbol Connector:Conn_01x04_Male
- added J7: USB C Connector, Connector_USB:USB_C_Receptacle_Amphenol_12401548E4-2A, symbol Connector:USB_C_Receptacle
- renumbered J1 to J8, SW16 to SW14, SW17 to SW15, SW14 to SW16, SW15 to SW17
Connections:
- net GND: now also J8.AGND, J8.GND@1 (GND), J8.GND@2 (GND), J8.GND@3 (GND), J8.GND@4 (GND), J8.GND@5 (GND), J8.GND@6 (GND), J8.GND@7 (GND), J8.GND@8 (GND), SW1.1, SW10.1, SW11.1, SW12.1, SW13.1, SW14.1, SW15.1, SW16.1, SW17.1, SW18.1, SW19.1, SW2.1, SW20.1, SW3.1, SW4.1, SW5.1, J1.1 (Pin_1), J10.1 (Pin_1), J11.1 (Pin_1), J12.1 (Pin_1), J2.1 (Pin_1), J3.1 (Pin_1), J4.1 (Pin_1), J5.1 (Pin_1), J5.2 (Pin_2), J6.1 (Pin_1), J7.A1 (GND), J7.A12 (GND), J7.B1 (GND), J7.B12 (GND), J7.S1 (SHIELD), J9.1 (Pin_1)
- net C_RT: now reaches SW20.2
- net C_RT: now also J4.6 (Pin_6)
- net M2: now reaches SW15.2
- net M2: now also J3.3 (Pin_3)
- net DOWN: now reaches SW8.2
- net DOWN: now also J1.3 (Pin_3)
- net LEFT: now reaches SW7.2
- net LEFT: now also J1.4 (Pin_4)
- net P START: now reaches J8.GP0
- net P C_UP: now reaches J8.GP12
- net P C_UP: now also J11.2 (Pin_2)
- net P C_LT: now reaches J8.GP13
- net P C_LT: now also J11.3 (Pin_3)
- net P A: now reaches J8.GP14
- net P A: now also J11.4 (Pin_4)
- net P C_DN: now reaches J8.GP15
- net P C_DN: now also J11.5 (Pin_5)
- net P C_RT: now reaches J8.GP16
- net P C_RT: now also J11.6 (Pin_6)
- net P UP: now reaches J8.GP17
- net P UP: now also J12.2 (Pin_2)
- net P MS: now reaches J8.GP18
- net P MS: now also J12.3 (Pin_3)
- net P Z: now reaches J8.GP19
- net P Z: now also J12.4 (Pin_4)
- net P RIGHT: now reaches J8.GP2
- net P RIGHT: now also J9.2 (Pin_2)
- net P LS: now reaches J8.GP20
- net P LS: now also J12.5 (Pin_5)
- net P X: now reaches J8.GP21
- net P X: now also J12.6 (Pin_6)
- net P Y: now reaches J8.GP22
- net P Y: now also J12.7 (Pin_7)
- net P B: now reaches J8.GP26_A0
- net P B: now also J12.8 (Pin_8)
- net P R: now reaches J8.GP27_A1
- net P R: now also J12.9 (Pin_9)
- net DATA: now reaches J8.GP28_A2
- net DATA: now also J5.4 (Pin_4), J7.A11 (RX2+), J7.B11 (RX1+)
- net P DOWN: now reaches J8.GP3
- net P DOWN: now also J9.3 (Pin_3)
- net P LEFT: now reaches J8.GP4
- net P LEFT: now also J9.4 (Pin_4)
- net P L: now reaches J8.GP5
- net P L: now also J9.5 (Pin_5)
- net P M1: now reaches J8.GP6
- net P M1: now also J10.2 (Pin_2)
- net P M2: now reaches J8.GP7
- net P M2: now also J10.3 (Pin_3)
- net D-: now reaches J8.TP2 (D+)
- net D-: now also J6.3 (Pin_3), J7.A7 (D-), J7.B7 (D-)
- net D+: now reaches J8.TP3 (D-)
- net D+: now also J6.2 (Pin_2), J7.A6 (D+), J7.B6 (D+)
- net +5V: now reaches J8.VBUS
- net +5V: now also J5.6 (Pin_6), J6.4 (Pin_4), J7.A4 (VBUS), J7.A9 (VBUS), J7.B4 (VBUS), J7.B9 (VBUS)
- net VCC: now reaches J8.VSYS
- net VCC: now also D1.1 (K), D2.1 (K), J5.3 (Pin_3)
- net Z: now reaches SW12.2
- net Z: now also J2.4 (Pin_4)
- net B: now reaches SW10.2
- net B: now also J2.8 (Pin_8)
- net Y: now reaches SW2.2
- net Y: now also J2.7 (Pin_7)
- net L: now reaches SW6.2
- net L: now also J1.5 (Pin_5)
- net X: now reaches SW11.2
- net X: now also J2.6 (Pin_6)
- net LS: now reaches SW3.2
- net LS: now also J2.5 (Pin_5)
- net R: now reaches SW1.2
- net R: now also J2.9 (Pin_9)
- net UP: now reaches SW13.2
- net UP: now also J2.2 (Pin_2)
- net MS: now reaches SW4.2
- net MS: now also J2.3 (Pin_3)
- net RIGHT: now reaches SW9.2
- net RIGHT: now also J1.2 (Pin_2)
- net M1: now reaches SW14.2
- net M1: now also J3.2 (Pin_2)
- net C_DN: now reaches SW18.2
- net C_DN: now also J4.5 (Pin_5)
- net START: now reaches SW5.2
- net C_UP: now reaches SW17.2
- net C_UP: now also J4.2 (Pin_2)
- net A: now reaches SW19.2
- net A: now also J4.4 (Pin_4)
- net C_LT: now reaches SW16.2
- net C_LT: now also J4.3 (Pin_3)
- new net +3V3: D1.2 (A), D2.2 (A), J5.5 (Pin_5), J7.A2 (TX1+), J7.B2 (TX2+)
- no-connect marks 0 -> 18
Other:
- moved on the sheet: J8, SW1, SW10, SW11, SW12, SW13, SW14, SW15, SW16, SW17, SW18, SW19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

Commit message: Primera iteración de la PCB
Parts:
- added H1, H10, H11, H12, H13, H14, H15, H16, H2, H3, H4, H5, H6, H7, H8, H9: MountingHole, MountingHole:MountingHole_2.2mm_M2_DIN965, symbol Mechanical:MountingHole
- added H17, H18, H19, H20: Quark Logo, qw-v-logo:qw new logo silk + copper md, symbol Mechanical:MountingHole

Commit message: Moving rowards integrated version
Parts:
- removed D1: D_Small, Diode_THT:D_DO-41_SOD81_P10.16mm_Horizontal, symbol Device:D_Small
- removed H1, H10, H11, H12, H13, H14, H15, H16, H2, H3, H4, H5, H6, H7, H8, H9: MountingHole, MountingHole:MountingHole_2.2mm_M2_DIN965, symbol Mechanical:MountingHole
- removed H17, H18, H19, H20: Quark Logo, qw-v-logo:qw new logo silk + copper md, symbol Mechanical:MountingHole
- removed J1, J9: Left Stick, Connector_PinHeader_2.54mm:PinHeader_1x05_P2.54mm_Vertical, symbol Connector:Conn_01x05_Male
- removed J10, J3: Modifiers, Connector_PinHeader_2.54mm:PinHeader_1x03_P2.54mm_Vertical, symbol Connector:Conn_01x03_Male
- removed J11, J4: C Stick, Connector_PinHeader_2.54mm:PinHeader_1x06_P2.54mm_Vertical, symbol Connector:Conn_01x06_Male
- removed J12, J2: Buttons, Connector_PinHeader_2.54mm:PinHeader_1x09_P2.54mm_Vertical, symbol Connector:Conn_01x09_Male
- removed J6: Extra USB, Connector_PinHeader_2.54mm:PinHeader_1x04_P2.54mm_Vertical, symbol Connector:Conn_01x04_Male
- removed J8: RPI_PICO-TH, OF1PI:RPI_PICO_TH, symbol rpi_pico-th:RPI_PICO-TH
- added C1, C2, C3, C7: 1uF, Capacitor_SMD:C_0402_1005Metric, symbol Device:C_Small
- added C10, C11, C12, C13, C14, C17, C4, C5, C8, C9: 100nF, Capacitor_SMD:C_0402_1005Metric, symbol Device:C_Small
- added C15, C16: 22pF, Capacitor_SMD:C_0402_1005Metric, symbol Device:C_Small
- added C6: 10uF, Capacitor_SMD:C_0402_1005Metric, symbol Device:C_Small
- added J3: JTAG_TC2030, marbastlib-various:CON_TC2030_outlined, symbol marbastlib-various:JTAG_TC2030
- added R1, R2: 5.1k, Resistor_SMD:R_0402_1005Metric, symbol Device:R_Small
- added R3: 10k, Resistor_SMD:R_0402_1005Metric, symbol Device:R_Small
- added R4, R5: 27R, Resistor_SMD:R_0603_1608Metric, symbol Device:R_Small
- added R6, R7: 1k, Resistor_SMD:R_0402_1005Metric, symbol Device:R_Small
- added SW21: Boot, Button_Switch_SMD:SW_SPST_SKQG_WithStem, symbol Switch:SW_Push
- added U1: XC6206, Package_TO_SOT_SMD:SOT-23, symbol Regulator_Linear:XC6206PxxxMR
- added U2: USBLC6-2SC6, Package_TO_SOT_SMD:SOT-23-6, symbol Power_Protection:USBLC6-2SC6
- added U3: RP2040, qw-footprints:RP2040-QFN-56, symbol Sleep-lib:RP2040
- added U4: W25Q128JVS, Package_SO:SOIC-8_5.23x5.23mm_P1.27mm, symbol Memory_Flash:W25Q128JVS
- added Y1: 12MHz, Crystal:Crystal_SMD_3225-4Pin_3.2x2.5mm, symbol Device:Crystal_GND24_Small
- renumbered D2 to D1, J7 to J1, J5 to J2
Connections:
- net +3V3: now also C10.1, C11.1, C12.1, C13.1, C14.1, C17.1, C2.2, C6.1, C7.1, C8.1, C9.1, J3.1 (VCC), R3.1, U1.2 (VO), U3.1 (IOVDD), U3.10 (IOVDD), U3.22 (IOVDD), U3.33 (IOVDD), U3.42 (IOVDD), U3.43 (ADC_AVDD), U3.44 (VREG_VIN), U3.48 (USB_VDD), U3.49 (IOVDD), U4.8 (VCC)
- net +5V: now also C1.2, U1.3 (VI), U2.5 (VBUS)
- net A: now also U3.17 (GPIO14)
- net B: now also U3.38 (GPIO26/ADC0)
- net C_DN: now also U3.18 (GPIO15)
- net C_LT: now also U3.16 (GPIO13)
- net C_RT: now also U3.27 (GPIO16)
- net C_UP: now also U3.15 (GPIO12)
- net D+: now also R4.1, U2.4 (I/O2); no longer J1.A6 (D+), J1.B6 (D+)
- net D-: now also R5.1, U2.6 (I/O1); no longer J1.A7 (D-), J1.B7 (D-)
- net DATA: now also U3.40 (GPIO28/ADC2)
- net DOWN: now also U3.5 (GPIO3)
- net GND: now also C1.1, C10.2, C11.2, C12.2, C13.2, C14.2, C15.1, C16.1, C17.2, C2.1, C3.2, C4.2, C5.2, C6.2, C7.2, C8.2, C9.2, J3.5 (GND), R1.2, R2.2, SW21.1, U1.1 (GND), U2.2 (GND), U3.19 (TESTEN), U3.57 (GND), U4.4 (GND), Y1.2, Y1.4
- net L: now also U3.7 (GPIO5)
- net LEFT: now also U3.6 (GPIO4)
- net LS: now also U3.31 (GPIO20)
- net M1: now also U3.8 (GPIO6)
- net M2: now also U3.9 (GPIO7)
- net MS: now also U3.29 (GPIO18)
- net R: now also U3.39 (GPIO27/ADC1)
- net RIGHT: now also U3.4 (GPIO2)
- net START: now also U3.2 (GPIO0)
- net UP: now also U3.28 (GPIO17)
- net X: now also U3.32 (GPIO21)
- net Y: now also U3.34 (GPIO22)
- net Z: now also U3.30 (GPIO19)
- net at J1.A5 (CC1): now also R2.1
- net at J1.B5 (CC2): now also R1.1
- new net +1V1: C3.1, C4.1, C5.1, U3.23 (DVDD), U3.45 (VREG_VOUT), U3.50 (DVDD)
- new net CS: R7.2, U3.56 (QSPI_SS_N), U4.1 (~{CS})
- new net DBUS+: J1.A6 (D+), J1.B6 (D+), U2.3 (I/O2)
- new net DBUS-: J1.A7 (D-), J1.B7 (D-), U2.1 (I/O1)
- new net D_+: R4.2, U3.47 (D+)
- new net D_-: R5.2, U3.46 (D-)
- new net QSPI_CLK: U3.52 (QSPI_SCLK), U4.6 (CLK)
- new net SD0: U3.53 (QSPI_SD0), U4.5 (DI(IO0))
- new net SD1: U3.55 (QSPI_SD1), U4.2 (DO(IO1))
- new net SD2: U3.54 (QSPI_SD2), U4.3 (IO2)
- new net SD3: U3.51 (QSPI_SD3), U4.7 (IO3)
- new net SWCLK: J3.4 (SWCLK), U3.24 (SWCLK)
- new net SWD: J3.2 (SWDIO), U3.25 (SWDIO)
- new net XTAL_IN: C15.2, U3.20 (XTAL_IN), Y1.3
- new net XTAL_O: C16.2, R6.1, Y1.1
- new net XTAL_OUT: R6.2, U3.21 (XTAL_OUT)
- new net ~{RESET}: J3.3 (~{RST}), R3.2, U3.26 (~{RUN})
- new net ~{USB_BOOT}: R7.1, SW21.2
- no-connect marks 18 -> 13
Other:
- moved on the sheet: D1, J1, J2

Commit message: Holy shit man
Parts:
- removed J2: GCC Cable, Connector_PinHeader_2.54mm:PinHeader_1x06_P2.54mm_Vertical, symbol Connector:Conn_01x06_Female
- added F1: Fuse_Small, Fuse:Fuse_1206_3216Metric, symbol Device:Fuse_Small
- D1: value D_Small -> Schottky Diode; footprint Diode_SMD:D_0805_2012Metric -> qw-footprints:CUSTOM D_SOD-123; LCSC (none) -> C130880
- J1: footprint Connector_USB:USB_C_Receptacle_Amphenol_12401548E4-2A -> qw-footprints:TYPE-C_24P_QCHT; LCSC (none) -> C456013
Connections:
- net +5V: now also F1.2; no longer J1.A4 (VBUS), J1.A9 (VBUS), J1.B4 (VBUS), J1.B9 (VBUS)
- net D+: now also U2.6 (I/O1); no longer U2.4 (I/O2)
- net D-: now also U2.4 (I/O2); no longer U2.6 (I/O1)
- net DBUS+: now also U2.1 (I/O1); no longer U2.3 (I/O2)
- net DBUS-: now also U2.3 (I/O2); no longer U2.1 (I/O1)
- new net: F1.1, J1.A4 (VBUS), J1.A9 (VBUS), J1.B4 (VBUS), J1.B9 (VBUS)

Commit message: WE REACHED SOMETHING
Parts:
- removed R1, R2: 5.1k, Resistor_SMD:R_0402_1005Metric, symbol Device:R_Small
- added SW12, SW14, SW15, SW18, SW2, SW20, SW21, SW24, SW25, SW27, SW30, SW31, SW33, SW36, SW37, SW4, SW40, SW6, SW8, SW9: MX_SW_solder, marbastlib-mx:SW_MX_1u, symbol marbastlib-mx:MX_SW_solder
- renumbered J3 to J2, SW5 to SW1, SW9 to SW10, SW1 to SW11, SW2 to SW13, SW3 to SW16, SW4 to SW17, SW10 to SW19, SW11 to SW22, SW12 to SW23, SW13 to SW26, SW14 to SW28, SW15 to SW29, SW6 to SW3, SW16 to SW32, SW17 to SW34, SW18 to SW35, SW19 to SW38, SW20 to SW39, SW21 to SW41, SW7 to SW5, SW8 to SW7
Connections:
- net A: now also U3.16 (GPIO13), SW37.1; no longer U3.17 (GPIO14)
- net B: now also SW20.1
- net C_DN: now also U3.17 (GPIO14), SW36.1; no longer U3.18 (GPIO15)
- net C_LT: now also U3.15 (GPIO12), SW31.1; no longer U3.16 (GPIO13)
- net C_RT: now also U3.18 (GPIO15), SW40.1; no longer U3.27 (GPIO16)
- net C_UP: now also U3.27 (GPIO16), SW33.1; no longer U3.15 (GPIO12)
- net DOWN: now also SW8.1
- net GND: now also SW12.2, SW14.2, SW15.2, SW18.2, SW2.2, SW20.2, SW21.2, SW24.2, SW25.2, SW27.2, SW30.2, SW31.2, SW33.2, SW36.2, SW37.2, SW4.2, SW40.2, SW6.2, SW8.2, SW9.2
- net L: now also SW4.1
- net LEFT: now also SW6.1
- net LS: now also SW15.1
- net M1: now also SW27.1
- net M2: now also SW30.1
- net MS: now also SW18.1
- net R: now also SW12.1
- net RIGHT: now also SW9.1
- net START: now also SW2.1
- net UP: now also SW25.1
- net VCC: now also F1.1, J1.A4 (VBUS), J1.A9 (VBUS), J1.B4 (VBUS), J1.B9 (VBUS)
- net X: now also SW21.1
- net Y: now also SW14.1
- net Z: now also SW24.1
- no-connect marks 13 -> 15
Other:
- moved on the sheet: SW1, SW10, SW19, SW22, SW23, SW26, SW28, SW29, SW3, SW35, SW38, SW39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

Commit message: Primera revisión
Parts:
- added D2: Schottky Diode, qw-footprints:CUSTOM D_SOD-123, symbol Device:D_Small
- added H1, H2, H3, H4, H5, H6, H7, H8: MountingHole, MountingHole:MountingHole_2.2mm_M2_ISO14580_Pad, symbol Mechanical:MountingHole
- renumbered C2 to C1, C1 to C2, R3 to R1, R4 to R2, R5 to R3, R6 to R4, R7 to R5
Connections:
- net +3V3: now also D1.1 (K), D2.1 (K); no longer D1.2 (A), J1.A2 (TX1+), J1.B2 (TX2+), U1.2 (VO)
- net VCC: no longer D1.1 (K)
- new net: D2.2 (A), U1.2 (VO)
- new net 3vCable: D1.2 (A), J1.A2 (TX1+), J1.B2 (TX2+)
Other:
- moved on the sheet: C1, C2, D1, U1

Commit message: Primera revisión + modelo
Parts:
- added H10, H9: MountingHole, MountingHole:MountingHole_2.2mm_M2_ISO14580_Pad, symbol Mechanical:MountingHole
- added H11: Logo, qw-logo:qw new logo mask md, symbol Mechanical:MountingHole
Changed lines of the file:
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@@
     (pin "2")
+  )
+  (symbol (lib_id "Mechanical:MountingHole") (at 139.8778 80.01 0) (unit 1)
+    (in_bom yes) (on_board yes) (fields_autoplaced)
+    (property "Reference" "H10" (id 0) (at 143.5354 78.7399 0)
+      (effects (font (size 1.27 1.27)) (justify left))
+    )
+    (property "Value" "MountingHole" (id 1) (at 143.5354 81.2799 0)
+      (effects (font (size 1.27 1.27)) (justify left))
+    )
+    (property "Footprint" "MountingHole:MountingHole_2.2mm_M2_ISO14580_Pad" (id 2) (at 139.8778 80.01 0)
+      (effects (font (size 1.27 1.27)) hide)
+    )
+    (property "Datasheet" "~" (id 3) (at 139.8778 80.01 0)
+      (effects (font (size 1.27 1.27)) hide)
+    )
   )
   (symbol (lib_id "marbastlib-mx:MX_SW_solder") (at 168.529 53.6956 180) (unit 1)
@@
     (pin "1")
     (pin "2")
+  )
+  (symbol (lib_id "Mechanical:MountingHole") (at 113.7666 98.298 0) (unit 1)
+    (in_bom yes) (on_board yes) (fields_autoplaced)
+    (property "Reference" "H11" (id 0) (at 117.4242 97.0279 0)
+      (effects (font (size 1.27 1.27)) (justify left))
+    )
+    (property "Value" "Logo" (id 1) (at 117.4242 99.5679 0)
+      (effects (font (size 1.27 1.27)) (justify left))
+    )
+    (property "Footprint" "qw-logo:qw new logo mask md" (id 2) (at 113.7666 98.298 0)
+      (effects (font (size 1.27 1.27)) hide)
+    )
+    (property "Datasheet" "~" (id 3) (at 113.7666 98.298 0)
+      (effects (font (size 1.27 1.27)) hide)
+    )
   )
   (symbol (lib_id "marbastlib-mx:MX_SW_solder") (at 228.4476 42.926 180) (unit 1)
@@
     (pin "2")
   )
+  (symbol (lib_id "Mechanical:MountingHole") (at 139.8778 74.4474 0) (unit 1)
+    (in_bom yes) (on_board yes) (fields_autoplaced)
+    (property "Reference" "H9" (id 0) (at 143.5354 73.1773 0)
+      (effects (font (size 1.27 1.27)) (justify left))
+    )
+    (property "Value" "MountingHole" (id 1) (at 143.5354 75.7173 0)
+      (effects (font (size 1.27 1.27)) (justify left))
+    )
+    (property "Footprint" "MountingHole:MountingHole_2.2mm_M2_ISO14580_Pad" (id 2) (at 139.8778 74.4474 0)
+      (effects (font (size 1.27 1.27)) hide)
+    )
+    (property "Datasheet" "~" (id 3) (at 139.8778 74.4474 0)
+      (effects (font (size 1.27 1.27)) hide)
+    )
+  )
   (symbol (lib_id "Device:C_Small") (at 233.5784 112.1664 0) (unit 1)
     (in_bom yes) (on_board yes)
@@
       (reference "H8") (unit 1) (value "MountingHole") (footprint "MountingHole:MountingHole_2.2mm_M2_ISO14580_Pad")
     )
+    (path "/db066b72-7f0e-4f77-a777-1e665b13cf49"
+      (reference "H9") (unit 1) (value "MountingHole") (footprint "MountingHole:MountingHole_2.2mm_M2_ISO14580_Pad")
+    )
+    (path "/02ab43e6-a8e8-44a2-9f11-9d4436e29bb7"
+      (reference "H10") (unit 1) (value "MountingHole") (footprint "MountingHole:MountingHole_2.2mm_M2_ISO14580_Pad")
+    )
+    (path "/3eb265a0-8ca3-424b-9513-7ff1b6d8e390"
+      (reference "H11") (unit 1) (value "Logo") (footprint "qw-logo:qw new logo mask md")
+    )
     (path "/a0fbf1f0-f019-47ec-af8b-330833a71f51"
